File: Board Files/WirelessTransceiverUSB_Rev-.brd (EAGLE design)
At the start: 33 x 55.9 mm, 37 parts, among them J1 MINI-USB-32005-201, U1 ATMEGA328PB-AU, U2 ADP121-AUJZ33R7, U3 FT230XS, Y2 CSTNE16M0V530000R0

Commit message: Corrected .brd file
Parts:
- moved C8 87.3 mm to (21.3, 2.29), turned to 90 degrees
- moved C7 83.1 mm to (15.5, 2.29), turned to 90 degrees
- moved C3 82.9 mm to (12.4, 2.29), turned to 90 degrees
- moved R10 82.9 mm to (15.0, -6.10), turned to 180 degrees
- moved R11 79.3 mm to (15.0, -8.64)
- moved R13 78.1 mm to (26.2, -5.59), turned to 180 degrees
- moved R12 76.9 mm to (26.2, -8.64), turned to 180 degrees
- moved C9 76.2 mm to (15.0, -10.9), turned to 180 degrees
- moved C10 76.2 mm to (15.0, -3.81), turned to 180 degrees
- moved C6 72.1 mm to (18.5, 2.29), turned to 90 degrees
- moved U3 68.9 mm to (20.3, -7.62), turned to 90 degrees
- moved RX 59.9 mm to (28.7, -30.5), turned to 180 degrees
- moved TX 56.0 mm to (28.7, -33.3), turned to 180 degrees
- moved L1 54.7 mm to (14.0, -1.27)
- moved R2 43.6 mm to (24.6, -30.5)
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Routing:
- net N$14: track 0.00 -> 31.0 mm, vias 0 -> 2
- net N$13: track 0.00 -> 27.2 mm, vias 0 -> 2
- net 3V3: track 14.0 -> 29.0 mm
- net 5V0: track 61.4 -> 75.9 mm, vias 5 -> 6
- net N$11: track 0.00 -> 13.2 mm, vias 0 -> 2
- net USBD_P: track 0.00 -> 12.0 mm
- net USBD_N: track 0.00 -> 11.5 mm
- net N$16: track 0.00 -> 9.18 mm, vias 0 -> 2
- net N$15: track 0.00 -> 8.56 mm, vias 0 -> 2
- net VBUS: track 5.48 -> 10.4 mm
- net N$4: track 0.00 -> 2.06 mm
- net N$1: track 0.00 -> 2.06 mm
- net TX: track 37.2 -> 38.5 mm
- net RX: track 33.6 -> 34.8 mm
- net D_N: track 7.35 -> 8.26 mm
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